Commit message: Added Camera link and changed world configuration

File: gantry/urdf/Gantry.urdf (robot description, URDF)
Before this commit: robot gantry, 7 links, 6 joints
Links:
- added link camera_link, mass 1e-5; collision box size=0.01 0.01 0.01; visual box size=0.01 0.01 0.01
Joints:
- added joint camera_joint: type fixed, parent world, child camera_link, origin xyz=1.8 -0.375 1.0 rpy=0 1.5708 0, axis 0 1 0

Commit message: Added Laser sensor for depth calculation and detect an object, changed colour of the robot

File: gantry/urdf/Gantry.urdf (robot description, URDF)
Before this commit: robot gantry, 8 links, 7 joints
Links:
- added link cam_on_laser_link, mass 1e-5; collision box size=0.01 0.01 0.01; visual box size=0.01 0.01 0.01
- added link laser_link, mass 1e-5; collision box size=0.01 0.01 0.01; visual box size=0.01 0.01 0.01
- link Cup: geometry collision mesh filename=package://gantry/meshes/Cup.dae; visual mesh filename=package://gantry/meshes/Cup.dae
- link X_Motion: geometry collision mesh filename=package://gantry/meshes/X_Motion.dae; visual mesh filename=package://gantry/meshes/X_Motion.dae
- link Y_Motion: geometry collision mesh filename=package://gantry/meshes/Y_Motion.dae; visual mesh filename=package://gantry/meshes/Y_Motion.dae
- link Z_Motion: geometry collision mesh filename=package://gantry/meshes/Z_Motion.dae; visual mesh filename=package://gantry/meshes/Z_Motion.dae
- link Z_Rot: geometry collision mesh filename=package://gantry/meshes/Z_Rot.dae; visual mesh filename=package://gantry/meshes/Z_Rot.dae
- link base_link: geometry collision mesh filename=package://gantry/meshes/base_link.dae; visual mesh filename=package://gantry/meshes/base_link.dae
Joints:
- added joint cam_on_laser_joint: type fixed, parent world, child cam_on_laser_link, origin xyz=1.8 -0.75 0.7 rpy=0 0 1.5708, axis 0 1 0
- added joint laser_joint: type fixed, parent world, child laser_link, origin xyz=1 -0.375 1.0 rpy=0 1.5708 0, axis 0 1 0

Commit message: Changed robot coordinate transformation frame

File: gantry/urdf/Gantry.urdf (robot description, URDF)
Before this commit: robot gantry, 10 links, 9 joints
Joints:
- joint X_Joint: origin xyz=-0.3 0.05 0.195 rpy=1.5708 0 1.5708 -> xyz=-0.05 0.05 1.095 rpy=1.5708 0 1.5708
- joint Y_Joint: origin xyz=0.1 0 0.21 rpy=0 -1.5708 0 -> xyz=0.035 0.2 -0.017 rpy=0 -1.5708 0
- joint Z_Joint: origin xyz=-0.0115 1.1071 0.19185 rpy=-1.5708 0 0 -> xyz=0.143 0.14 0.12685 rpy=-1.5708 0 0
- joint Z_Rot_Joint: origin xyz=0.25743 0 0.0031492 rpy=0 0 0 -> xyz=0.08 0 -0.14 rpy=0 0 0

Commit message: Added Output boxes and conveyor, collision checking done

File: gantry/urdf/Gantry.urdf (robot description, URDF)
Before this commit: robot gantry, 10 links, 9 joints
Joints:
- joint X_Joint: limit lower=-0.45 upper=0.48 effort=20 velocity=1 -> lower=-0.5 upper=0.5 effort=20 velocity=1
- joint cam_on_laser_joint: origin xyz=1.8 -0.75 0.7 rpy=0 0 1.5708 -> xyz=1.8 -0.75 0.62 rpy=0 0 1.5708

File: gantry/urdf/conveyor2.urdf (robot description, URDF)
Before this commit: robot conveyor_belt, 3 links, 2 joints
Links:
- added link Big_box, mass 0.0020128; collision mesh filename=package://gantry/meshes/Big_box.dae; visual mesh filename=package://gantry/meshes/Big_box.dae
- added link Big_box2, mass 0.0020128; collision mesh filename=package://gantry/meshes/Big_box.dae; visual mesh filename=package://gantry/meshes/Big_box.dae
Joints:
- added joint Big_box_Joint: type fixed, parent world, child Big_box, origin xyz=0.4 0.325 0.69 rpy=0 -1.5708 1.5708, axis 0 0 1
- added joint Big_box_Joint2: type fixed, parent world, child Big_box2, origin xyz=-0.275 0.325 0.69 rpy=0 -1.5708 1.5708, axis 0 0 1
- joint fixed: origin xyz=0.9 -0.375 0.0 rpy=0.0 0.0 -1.5708 -> xyz=0.9 0.325 0.0 rpy=0.0 0.0 -1.5708

Commit message: Stopping added

File: gantry/urdf/Gantry.urdf (robot description, URDF)
Before this commit: robot gantry, 10 links, 9 joints
Joints:
- joint laser_joint: origin xyz=1 -0.375 1.0 rpy=0 1.5708 0 -> xyz=1.75 -0.375 1.0 rpy=0 1.5708 0

Commit message: incomplete working of picking

File: gantry/urdf/Gantry.urdf (robot description, URDF)
Before this commit: robot gantry, 10 links, 9 joints
Links:
- link Cup: geometry collision mesh filename=package://gantry/meshes/Cup1.dae; visual mesh filename=package://gantry/meshes/Cup1.dae
- link Z_Rot: geometry collision mesh filename=package://gantry/meshes/onlyrod.dae; visual mesh filename=package://gantry/meshes/onlyrod.dae
Joints:
- joint Cup_Joint: limit (none) -> lower=-3.14 upper=3.14 effort=5 velocity=1; origin xyz=-0.0 -0.05 -0.48 rpy=3.1416 -0.0 0 -> xyz=-0.0 -0.002 -0.50 rpy=3.1416 -0.0 0; type fixed -> revolute
- joint Z_Rot_Joint: origin xyz=0.08 0 -0.14 rpy=0 0 0 -> xyz=0.08 -0.002 -0.14 rpy=0 0 0

Commit message: Picking issue solved, placing issue remaining

File: gantry/urdf/Gantry.urdf (robot description, URDF)
Before this commit: robot gantry, 10 links, 9 joints
Joints:
- joint Cup_Joint: limit lower=-3.14 upper=3.14 effort=5 velocity=1 -> lower=-3.14 upper=3.14 effort=5 velocity=0

Commit message: Latest code

File: gantry/urdf/Gantry.urdf (robot description, URDF)
Before this commit: robot gantry, 10 links, 9 joints
Links:
- link Cup: mass 0.0020128 -> 0.050128
Joints:
- joint Cup_Joint: origin xyz=-0.0 -0.002 -0.50 rpy=3.1416 -0.0 0 -> xyz=0.0 -0.0015 -0.5 rpy=3.1416 -0.0 0

File: gantry/urdf/Gantry_copy.urdf (robot description, URDF)
Before this commit: robot gantry, 10 links, 9 joints
Joints:
- joint Cup_Joint: limit (none) -> lower=-0 upper=0 effort=5 velocity=0; type continuous -> revolute

File: gantry/urdf/conveyor2.urdf (robot description, URDF)
Before this commit: robot conveyor_belt2, 5 links, 4 joints
Links:
- link Big_box: mass 0.0020128 -> 20.128; geometry visual mesh filename=package://gantry/meshes/Big_box.dae
- link Big_box2: mass 0.0020128 -> 20.128; geometry visual mesh filename=package://gantry/meshes/Big_box.dae
